File: Inductor_Saturation_Tester-KiCAD/Logic.kicad_sch (KiCad schematic)
At the start: 13 parts, among them Q3 MMBT3904, Q4 MMBT3904, Q5 MMBT3906, Q6 MMBT3904, Q7 MMBT3904, Q8 MMBT3906, SW1 SW_MEC_5E, U6 NE555D

Commit message: update Rev B
Parts:
- removed Q3, Q4, Q6, Q7: MMBT3904, Package_TO_SOT_SMD:SOT-23, symbol Transistor_BJT:MMBT3904
- removed Q5, Q8: MMBT3906, Package_TO_SOT_SMD:SOT-23, symbol Transistor_BJT:MMBT3906
- added Q3, Q5, Q6, Q8: DMN67D7L, Package_TO_SOT_SMD:SOT-23, symbol Transistor_FET:DMN67D7L
- added Q4, Q7: BSS84, Package_TO_SOT_SMD:SOT-23, symbol Transistor_FET:BSS84
Connections:
- net +5VP: now also Q4.2 (S), Q7.2 (S)
- net GND: now also Q3.2 (S), Q5.2 (S), Q6.2 (S), Q8.2 (S)
- net NMOS_Gate: now also Q4.3 (D), Q5.3 (D)
- net PMOS_Gate: now also Q7.3 (D), Q8.3 (D)
- net TurnOn: now also Q4.1 (G), Q5.1 (G), Q6.1 (G)
- net at C7.1, R15.1: now also Q3.1 (G)
- net at R16.1, SW1.1, SW1.2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: now also Q3.3 (D)
- net at R17.1: now also Q6.3 (D), Q7.1 (G), Q8.1 (G)
Changed lines of the file:
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@@
     )
-  )
-  (symbol (lib_id "Transistor_BJT:MMBT3904") (at 199.39 39.37 0) (unit 1)
-    (in_bom yes) (on_board yes)
-    (property "Reference" "Q4" (id 0) (at 204.2414 38.2016 0)
-      (effects (font (size 1.27 1.27)) (justify left))
-    )
-    (property "Value" "MMBT3904" (id 1) (at 204.2414 40.513 0)
-      (effects (font (size 1.27 1.27)) (justify left))
-    )
-    (property "Footprint" "Package_TO_SOT_SMD:SOT-23" (id 2) (at 204.47 41.275 0)
-      (effects (font (size 1.27 1.27) italic) (justify left) hide)
-    )
-    (property "Datasheet" "https://www.onsemi.com/pub/Collateral/2N3903-D.PDF" (id 3) (at 199.39 39.37 0)
-      (effects (font (size 1.27 1.27)) (justify left) hide)
-    )
-    (pin "1")
-    (pin "2")
-    (pin "3")
-  )
-  (symbol (lib_id "Transistor_BJT:MMBT3906") (at 199.39 59.69 0) (mirror x) (unit 1)
-    (in_bom yes) (on_board yes)
-    (property "Reference" "Q5" (id 0) (at 204.2414 58.5216 0)
-      (effects (font (size 1.27 1.27)) (justify left))
-    )
-    (property "Value" "MMBT3906" (id 1) (at 204.2414 60.833 0)
-      (effects (font (size 1.27 1.27)) (justify left))
-    )
-    (property "Footprint" "Package_TO_SOT_SMD:SOT-23" (id 2) (at 204.47 57.785 0)
-      (effects (font (size 1.27 1.27) italic) (justify left) hide)
-    )
-    (property "Datasheet" "https://www.onsemi.com/pub/Collateral/2N3906-D.PDF" (id 3) (at 199.39 59.69 0)
-      (effects (font (size 1.27 1.27)) (justify left) hide)
-    )
-    (pin "1")
-    (pin "2")
-    (pin "3")
-  )
-  (symbol (lib_id "Transistor_BJT:MMBT3904") (at 66.04 60.96 0) (unit 1)
-    (in_bom yes) (on_board yes)
-    (property "Reference" "Q3" (id 0) (at 70.8914 59.7916 0)
-      (effects (font (size 1.27 1.27)) (justify left))
-    )
-    (property "Value" "MMBT3904" (id 1) (at 70.8914 62.103 0)
-      (effects (font (size 1.27 1.27)) (justify left))
-    )
-    (property "Footprint" "Package_TO_SOT_SMD:SOT-23" (id 2) (at 71.12 62.865 0)
-      (effects (font (size 1.27 1.27) italic) (justify left) hide)
-    )
-    (property "Datasheet" "https://www.onsemi.com/pub/Collateral/2N3903-D.PDF" (id 3) (at 66.04 60.96 0)
-      (effects (font (size 1.27 1.27)) (justify left) hide)
-    )
-    (pin "1")
-    (pin "2")
-    (pin "3")
   )
   (symbol (lib_id "Device:R") (at 48.26 60.96 270) (unit 1)
@@
     (pin "1")
   )
-  (symbol (lib_id "Transistor_BJT:MMBT3904") (at 199.39 97.79 0) (unit 1)
-    (in_bom yes) (on_board yes)
-    (property "Reference" "Q6" (id 0) (at 204.2414 96.6216 0)
-      (effects (font (size 1.27 1.27)) (justify left))
-    )
-    (property "Value" "MMBT3904" (id 1) (at 204.2414 98.933 0)
-      (effects (font (size 1.27 1.27)) (justify left))
-    )
-    (property "Footprint" "Package_TO_SOT_SMD:SOT-23" (id 2) (at 204.47 99.695 0)
-      (effects (font (size 1.27 1.27) italic) (justify left) hide)
-    )
-    (property "Datasheet" "https://www.onsemi.com/pub/Collateral/2N3903-D.PDF" (id 3) (at 199.39 97.79 0)
-      (effects (font (size 1.27 1.27)) (justify left) hide)
-    )
-    (pin "1")
-    (pin "2")
-    (pin "3")
-  )
   (symbol (lib_id "power:+5VP") (at 201.93 77.47 0) (unit 1)
     (in_bom yes) (on_board yes)
@@
     )
     (pin "1")
-  )
-  (symbol (lib_id "Transistor_BJT:MMBT3904") (at 240.03 81.28 0) (unit 1)
-    (in_bom yes) (on_board yes)
-    (property "Reference" "Q7" (id 0) (at 244.8814 80.1116 0)
-      (effects (font (size 1.27 1.27)) (justify left))
-    )
-    (property "Value" "MMBT3904" (id 1) (at 244.8814 82.423 0)
-      (effects (font (size 1.27 1.27)) (justify left))
-    )
-    (property "Footprint" "Package_TO_SOT_SMD:SOT-23" (id 2) (at 245.11 83.185 0)
-      (effects (font (size 1.27 1.27) italic) (justify left) hide)
-    )
-    (property "Datasheet" "https://www.onsemi.com/pub/Collateral/2N3903-D.PDF" (id 3) (at 240.03 81.28 0)
-      (effects (font (size 1.27 1.27)) (justify left) hide)
-    )
-    (pin "1")
-    (pin "2")
-    (pin "3")
-  )
-  (symbol (lib_id "Transistor_BJT:MMBT3906") (at 240.03 101.6 0) (mirror x) (unit 1)
-    (in_bom yes) (on_board yes)
-    (property "Reference" "Q8" (id 0) (at 244.8814 100.4316 0)
-      (effects (font (size 1.27 1.27)) (justify left))
-    )
-    (property "Value" "MMBT3906" (id 1) (at 244.8814 102.743 0)
-      (effects (font (size 1.27 1.27)) (justify left))
-    )
-    (property "Footprint" "Package_TO_SOT_SMD:SOT-23" (id 2) (at 245.11 99.695 0)
-      (effects (font (size 1.27 1.27) italic) (justify left) hide)
-    )
-    (property "Datasheet" "https://www.onsemi.com/pub/Collateral/2N3906-D.PDF" (id 3) (at 240.03 101.6 0)
-      (effects (font (size 1.27 1.27)) (justify left) hide)
-    )
-    (pin "1")
-    (pin "2")
-    (pin "3")
   )
   (symbol (lib_id "power:GND") (at 242.57 106.68 0) (unit 1)
@@
     (pin "1")
   )
+  (symbol (lib_id "Transistor_FET:BSS84") (at 240.03 81.28 0) (mirror x) (unit 1)
+    (in_bom yes) (on_board yes) (fields_autoplaced)
+    (property "Reference" "Q7" (id 0) (at 245.237 80.3715 0)
+      (effects (font (size 1.27 1.27)) (justify left))
+    )
+    (property "Value" "BSS84" (id 1) (at 245.237 83.1466 0)
+      (effects (font (size 1.27 1.27)) (justify left))
+    )
+    (property "Footprint" "Package_TO_SOT_SMD:SOT-23" (id 2) (at 245.11 79.375 0)
+      (effects (font (size 1.27 1.27) italic) (justify left) hide)
+    )
+    (property "Datasheet" "http://assets.nexperia.com/documents/data-sheet/BSS84.pdf" (id 3) (at 240.03 81.28 0)
+      (effects (font (size 1.27 1.27)) (justify left) hide)
+    )
+    (pin "1")
+    (pin "2")
+    (pin "3")
+  )
   (symbol (lib_id "Device:C") (at 102.87 69.85 0) (unit 1)
     (in_bom yes) (on_board yes)
@@
     (pin "1")
     (pin "2")
+  )
+  (symbol (lib_id "Transistor_FET:DMN67D7L") (at 199.39 97.79 0) (unit 1)
+    (in_bom yes) (on_board yes) (fields_autoplaced)
+    (property "Reference" "Q6" (id 0) (at 204.597 96.8815 0)
+      (effects (font (size 1.27 1.27)) (justify left))
+    )
+    (property "Value" "DMN67D7L" (id 1) (at 204.597 99.6566 0)
+      (effects (font (size 1.27 1.27)) (justify left))
+    )
+    (property "Footprint" "Package_TO_SOT_SMD:SOT-23" (id 2) (at 204.47 99.695 0)
+      (effects (font (size 1.27 1.27) italic) (justify left) hide)
+    )
+    (property "Datasheet" "http://www.diodes.com/assets/Datasheets/DMN67D7L.pdf" (id 3) (at 199.39 97.79 0)
+      (effects (font (size 1.27 1.27)) (justify left) hide)
+    )
+    (pin "1")
+    (pin "2")
+    (pin "3")
+  )
+  (symbol (lib_id "Transistor_FET:DMN67D7L") (at 199.39 59.69 0) (unit 1)
+    (in_bom yes) (on_board yes) (fields_autoplaced)
+    (property "Reference" "Q5" (id 0) (at 204.597 58.7815 0)
+      (effects (font (size 1.27 1.27)) (justify left))
+    )
+    (property "Value" "DMN67D7L" (id 1) (at 204.597 61.5566 0)
+      (effects (font (size 1.27 1.27)) (justify left))
+    )
+    (property "Footprint" "Package_TO_SOT_SMD:SOT-23" (id 2) (at 204.47 61.595 0)
+      (effects (font (size 1.27 1.27) italic) (justify left) hide)
+    )
+    (property "Datasheet" "http://www.diodes.com/assets/Datasheets/DMN67D7L.pdf" (id 3) (at 199.39 59.69 0)
+      (effects (font (size 1.27 1.27)) (justify left) hide)
+    )
+    (pin "1")
+    (pin "2")
+    (pin "3")
+  )
+  (symbol (lib_id "Transistor_FET:DMN67D7L") (at 66.04 60.96 0) (unit 1)
+    (in_bom yes) (on_board yes) (fields_autoplaced)
+    (property "Reference" "Q3" (id 0) (at 71.247 60.0515 0)
+      (effects (font (size 1.27 1.27)) (justify left))
+    )
+    (property "Value" "DMN67D7L" (id 1) (at 71.247 62.8266 0)
+      (effects (font (size 1.27 1.27)) (justify left))
+    )
+    (property "Footprint" "Package_TO_SOT_SMD:SOT-23" (id 2) (at 71.12 62.865 0)
+      (effects (font (size 1.27 1.27) italic) (justify left) hide)
+    )
+    (property "Datasheet" "http://www.diodes.com/assets/Datasheets/DMN67D7L.pdf" (id 3) (at 66.04 60.96 0)
+      (effects (font (size 1.27 1.27)) (justify left) hide)
+    )
+    (pin "1")
+    (pin "2")
+    (pin "3")
   )
   (symbol (lib_id "power:GND") (at 95.25 96.52 0) (unit 1)
@@
     (pin "4")
   )
+  (symbol (lib_id "Transistor_FET:DMN67D7L") (at 240.03 101.6 0) (unit 1)
+    (in_bom yes) (on_board yes) (fields_autoplaced)
+    (property "Reference" "Q8" (id 0) (at 245.237 100.6915 0)
+      (effects (font (size 1.27 1.27)) (justify left))
+    )
+    (property "Value" "DMN67D7L" (id 1) (at 245.237 103.4666 0)
+      (effects (font (size 1.27 1.27)) (justify left))
+    )
+    (property "Footprint" "Package_TO_SOT_SMD:SOT-23" (id 2) (at 245.11 103.505 0)
+      (effects (font (size 1.27 1.27) italic) (justify left) hide)
+    )
+    (property "Datasheet" "http://www.diodes.com/assets/Datasheets/DMN67D7L.pdf" (id 3) (at 240.03 101.6 0)
+      (effects (font (size 1.27 1.27)) (justify left) hide)
+    )
+    (pin "1")
+    (pin "2")
+    (pin "3")
+  )
+  (symbol (lib_id "Transistor_FET:BSS84") (at 199.39 39.37 0) (mirror x) (unit 1)
+    (in_bom yes) (on_board yes) (fields_autoplaced)
+    (property "Reference" "Q4" (id 0) (at 204.597 38.4615 0)
+      (effects (font (size 1.27 1.27)) (justify left))
+    )
+    (property "Value" "BSS84" (id 1) (at 204.597 41.2366 0)
+      (effects (font (size 1.27 1.27)) (justify left))
+    )
+    (property "Footprint" "Package_TO_SOT_SMD:SOT-23" (id 2) (at 204.47 37.465 0)
+      (effects (font (size 1.27 1.27) italic) (justify left) hide)
+    )
+    (property "Datasheet" "http://assets.nexperia.com/documents/data-sheet/BSS84.pdf" (id 3) (at 199.39 39.37 0)
+      (effects (font (size 1.27 1.27)) (justify left) hide)
+    )
+    (pin "1")
+    (pin "2")
+    (pin "3")
+  )
 )
