File: Inductor_Saturation_Tester-KiCAD/Saturation_Tester.kicad_pcb (KiCad board)
At the start: 2 copper layers, 94.4 x 90 mm, 77 parts, among them J1 Conn_Coaxial, J10 Conn_Coaxial, J11 Screw_Terminal_01x03, J2 Conn_Coaxial, J3 Conn_Coaxial, J4 Conn_Coaxial, J5 Conn_Coaxial, J6 Barrel_Jack_Switch, J7 Conn_Coaxial, J8 Barrel_Jack_Switch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

Commit message: Rev B Update
Parts:
- removed BUF1: BUF634, Package_SO:SO-8_3.9x4.9mm_P1.27mm
- removed J1: Conn_Coaxial, Connector_Coaxial:BNC_TEConnectivity_1478204_Vertical
- removed R1, R10, R14, R2: 0, Resistor_SMD:R_1206_3216Metric
- removed R3, R4: DNP, Resistor_SMD:R_1206_3216Metric
- removed U1: LM358, Package_SO:SO-8_3.9x4.9mm_P1.27mm
- added C15: 10n, Capacitor_SMD:C_1206_3216Metric_Pad1.33x1.80mm_HandSolder, F.Cu at (99.5, 99.5)
- added C16: 100u, Capacitor_THT:CP_Radial_D8.0mm_P5.00mm, F.Cu at (120.2, 60.7)
- added C17: 100u, Capacitor_THT:CP_Radial_D8.0mm_P5.00mm, F.Cu at (102.0, 60.8)
- added C18: 100u, Capacitor_THT:CP_Radial_D8.0mm_P5.00mm, F.Cu at (111.0, 60.7)
- added C21: 100u, Capacitor_THT:CP_Radial_D8.0mm_P5.00mm, F.Cu at (103.6, 66.5)
- added C22: 100u, Capacitor_THT:CP_Radial_D8.0mm_P5.00mm, F.Cu at (94.3, 66.5)
- added C23: 100u, Capacitor_THT:CP_Radial_D8.0mm_P5.00mm, F.Cu at (83.8, 66.8)
- added C24: 100u, Capacitor_THT:CP_Radial_D8.0mm_P5.00mm, F.Cu at (89.3, 75.0)
- added R23: 22, Resistor_SMD:R_1206_3216Metric, F.Cu at (101.5, 82.7)
- added SW1: SW_MEC_5E, Eli_Lib:BigButton_TL1100F160Q, F.Cu at (129.5, 129.0)
- C1: value DNP -> 100u; footprint Capacitor_SMD:C_0805_2012Metric -> Capacitor_THT:CP_Radial_D8.0mm_P5.00mm
- C14, C19: value 100n -> 100u; footprint Capacitor_SMD:C_0805_2012Metric -> Capacitor_THT:CP_Radial_D8.0mm_P5.00mm
- C2: value DNP -> 100u; footprint Capacitor_SMD:C_0805_2012Metric -> Capacitor_THT:CP_Radial_D8.0mm_P5.00mm; moved to F.Cu
- C20: value 100n -> 100u; footprint Capacitor_SMD:C_0805_2012Metric -> Capacitor_THT:CP_Radial_D8.0mm_P5.00mm; moved to F.Cu
- C3: moved to B.Cu
- Q3, Q6: value MMBT3904 -> DMN67D7L
- Q4, Q7: value MMBT3904 -> BSS84
- Q5, Q8: value MMBT3906 -> DMN67D7L
- R11: value 100 -> DNP
- R24: value R -> 10m
- R8: value 270 -> 249
- moved C11 57.4 mm to (107.5, 80.8)
- moved C3 33.1 mm to (124.5, 99.0), turned to 0 degrees
- moved R22 32.1 mm to (87.3, 104.0), turned to 180 degrees
- moved C19 30.4 mm to (79.6, 75.2)
- moved C7 27.6 mm to (112.5, 107.5), turned to 180 degrees
- moved C12 27.2 mm to (131.0, 101.0), turned to 180 degrees
- moved C1 22.1 mm to (113.1, 66.5), turned to 0 degrees
- moved C14 14.9 mm to (91.5, 60.9), turned to 90 degrees
- moved Q6 14.4 mm to (123.0, 78.0), turned to 90 degrees
- moved Q7 12.5 mm to (123.0, 74.0), turned to 90 degrees
- moved U6 11.3 mm to (106.0, 101.4)
- moved R16 11.0 mm to (112.5, 99.0)
- moved C13 10.7 mm to (103.0, 105.0), turned to 180 degrees
- moved C2 10.4 mm to (108.2, 74.8), turned to 0 degrees
- moved Q3 9.84 mm to (112.0, 101.9)
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Connections:
- C1 pad 1: Net-(C1-Pad1) -> AltPower
- C14 pad 1: +5VP -> AltPower
- C19 pad 1: +5VP -> AltPower
- C2 pad 1: Net-(BUF1-Pad3) -> AltPower
- C2 pad 2: Net-(C2-Pad2) -> GND
- C20 pad 1: -5V -> AltPower
- D4 pad 1: +5VP -> AltPower
- D4 pad 2: RShunt- -> RShunt+
- J11 pad 3: Net-(J11-Pad3) -> InputLogic
- J7 pad 1: RShunt- -> RShunt+
- Q4 pad 2: NMOS_Gate -> +5VP
- Q4 pad 3: +5VP -> NMOS_Gate
- Q5 pad 2: NMOS_Gate -> GND
- Q5 pad 3: GND -> NMOS_Gate
- Q7 pad 2: PMOS_Gate -> +5VP
- Q7 pad 3: +5VP -> PMOS_Gate
- Q8 pad 2: PMOS_Gate -> GND
- Q8 pad 3: GND -> PMOS_Gate
- R11 pad 2: I_Return -> RShunt+
- R24 pad 1: I_Return -> RShunt+
- U4 pad 5: I_Return -> RShunt+
- U6 pad 6: Net-(U6-Pad6) -> unconnected-(U6-Pad6)
- U6 pad 7: Net-(U6-Pad7) -> unconnected-(U6-Pad7)
Routing:
- net +5VP: track 41.6 -> 192.4 mm, vias 2 -> 13
- net Net-(R18-Pad2): track 0.00 -> 68.5 mm, vias 0 -> 4
- net AltPower: track 0.00 -> 56.1 mm, vias 0 -> 2
- net Net-(R22-Pad1): track 0.00 -> 55.2 mm, vias 0 -> 2
- net RShunt-: track 0.00 -> 51.5 mm, vias 0 -> 2
- net InputLogic: track 0.00 -> 49.1 mm, vias 0 -> 3
- net Net-(R16-Pad1): track 0.00 -> 47.8 mm, vias 0 -> 2
- net RShunt+: track 0.00 -> 41.1 mm, vias 0 -> 15
- net TurnOn: track 0.00 -> 37.8 mm
- net -5V: track 30.7 -> 0.00 mm, vias 3 -> 0
- net Net-(C2-Pad2): track 28.4 -> 0.00 mm, vias 3 -> 0
- net IOut: track 1.41 -> 24.6 mm
- net I_Lim_Comp: track 0.00 -> 23.1 mm
- net Net-(C1-Pad1): track 21.2 -> 0.00 mm
- net Net-(R5-Pad1): track 0.00 -> 18.2 mm
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- added copper zone on B.Cu, net AltPower
- added copper zone on F.Cu, net AltPower
- added copper zone on F.Cu, net IOut
- added copper zone on B.Cu, net RShunt+
- added copper zone on F.Cu, net RShunt+
- added copper zone on F.Cu, net RShunt-
Other:
- net class Default removed
- board text added: "+5V"
- board text added: "Inductor Saturation Tester Rev B Eli Mattingly 23 AUG 2022"
- board text added: "Start Button"
- board text added: "Start Trig"
- board text removed: "+Vs"
- board text removed: "-Vs"
- board text removed: "BW"
- board text removed: "Impedance Analyzer Rev B Eli Mattingly 15 DEC 2021"
- board text removed: "Voltage Input"
