File: Inductor_Saturation_Tester-KiCAD/file6261FB5F.kicad_sch (KiCad schematic)
At the start: 39 parts, among them J6 Barrel_Jack_Switch, J8 Barrel_Jack_Switch, U2 LM358, U3 LM358, U4 LM358, U5 L7805

Commit message: update Rev B
Parts:
- gave numbers to parts that had none: 8
Changed lines of the file:
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@@
   (symbol (lib_id "Device:CP") (at 265.43 137.16 0) (unit 1)
     (in_bom yes) (on_board yes)
-    (property "Reference" "C?" (id 0) (at 268.4272 135.9916 0)
+    (property "Reference" "C24" (id 0) (at 268.4272 135.9916 0)
       (effects (font (size 1.27 1.27)) (justify left))
     )
@@
   (symbol (lib_id "Device:CP") (at 220.98 137.16 0) (unit 1)
     (in_bom yes) (on_board yes)
-    (property "Reference" "C?" (id 0) (at 223.9772 135.9916 0)
+    (property "Reference" "C19" (id 0) (at 223.9772 135.9916 0)
       (effects (font (size 1.27 1.27)) (justify left))
     )
@@
   (symbol (lib_id "Device:CP") (at 229.87 137.16 0) (unit 1)
     (in_bom yes) (on_board yes)
-    (property "Reference" "C?" (id 0) (at 232.8672 135.9916 0)
+    (property "Reference" "C20" (id 0) (at 232.8672 135.9916 0)
       (effects (font (size 1.27 1.27)) (justify left))
     )
@@
   (symbol (lib_id "power:GND") (at 238.76 154.94 0) (unit 1)
     (in_bom yes) (on_board yes)
-    (property "Reference" "#PWR?" (id 0) (at 238.76 161.29 0)
+    (property "Reference" "#PWR0102" (id 0) (at 238.76 161.29 0)
       (effects (font (size 1.27 1.27)) hide)
     )
@@
   (symbol (lib_id "Device:CP") (at 256.54 137.16 0) (unit 1)
     (in_bom yes) (on_board yes)
-    (property "Reference" "C?" (id 0) (at 259.5372 135.9916 0)
+    (property "Reference" "C23" (id 0) (at 259.5372 135.9916 0)
       (effects (font (size 1.27 1.27)) (justify left))
     )
@@
   (symbol (lib_id "Device:CP") (at 212.09 137.16 0) (unit 1)
     (in_bom yes) (on_board yes)
-    (property "Reference" "C?" (id 0) (at 215.0872 135.9916 0)
+    (property "Reference" "C2" (id 0) (at 215.0872 135.9916 0)
       (effects (font (size 1.27 1.27)) (justify left))
     )
@@
   (symbol (lib_id "power:GND") (at 203.2 154.94 0) (unit 1)
     (in_bom yes) (on_board yes)
-    (property "Reference" "#PWR?" (id 0) (at 203.2 161.29 0)
+    (property "Reference" "#PWR0101" (id 0) (at 203.2 161.29 0)
       (effects (font (size 1.27 1.27)) hide)
     )
@@
   (symbol (lib_id "Device:CP") (at 238.76 137.16 0) (unit 1)
     (in_bom yes) (on_board yes)
-    (property "Reference" "C?" (id 0) (at 241.7572 135.9916 0)
+    (property "Reference" "C21" (id 0) (at 241.7572 135.9916 0)
       (effects (font (size 1.27 1.27)) (justify left))
     )
@@
   (symbol (lib_id "Device:CP") (at 247.65 137.16 0) (unit 1)
     (in_bom yes) (on_board yes)
-    (property "Reference" "C?" (id 0) (at 250.6472 135.9916 0)
+    (property "Reference" "C22" (id 0) (at 250.6472 135.9916 0)
       (effects (font (size 1.27 1.27)) (justify left))
     )
@@
   (symbol (lib_id "Device:CP") (at 203.2 137.16 0) (unit 1)
     (in_bom yes) (on_board yes)
-    (property "Reference" "C?" (id 0) (at 206.1972 135.9916 0)
-      (effects (font (size 1.27 1.27)) (justify left))
-    )
+    (property "Reference" "C1" (id 0) (at 206.1972 135.9916 0)
+      (effects (font (size 1.27 1.27)) (justify left))
+    )
